File: UI.kicad_sch (KiCad schematic)
At the start: 40 parts, among them J501 RGB_OUT, Q501 AO3400A, SW501 BUTTON1, SW502 BUTTON2, SW503 BUTTON3, SW504 BUTTON4, SW505 BUTTON5, U501 74LVC1G34, U502 SSD1315 OLED 0.98"

Commit message: Started the checking of the components
Parts:
- BZ501, C501, C502, C503, C504, C505, C506, D501, D502, D503, D504, D505, D506, D507, D508, D509, D510, J501, JP501, JP502, R501, R502, R503, R504, R505, R506, R507, R508, R509, R510, R511, R512: Checked (none) -> OK

Commit message: Continued to check components footprints
Parts:
- Q501, U501: Checked (none) -> OK
- U502: Checked (none) -> E- Da Valutare
Changed lines of the file:
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@@
 			)
 		)
-		(property "Checked" ""
+		(property "Checked" "OK"
 			(at 46.99 38.1 0)
 			(effects
@@
 			)
 		)
-		(property "Checked" ""
+		(property "Checked" "E- Da Valutare"
 			(at 227.33 82.55 90)
 			(effects
@@
 			)
 		)
-		(property "Checked" ""
+		(property "Checked" "OK"
 			(at 163.83 86.36 0)
 			(effects

Commit message: Changed two connectors
Parts:
- U502: footprint Connector_PinHeader_1.00mm:PinHeader_1x04_P1.00mm_Vertical -> Connector_PinHeader_2.54mm:PinHeader_1x04_P2.54mm_Vertical
Changed lines of the file:
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@@
 			)
 		)
-		(property "Footprint" "Connector_PinHeader_1.00mm:PinHeader_1x04_P1.00mm_Vertical"
+		(property "Footprint" "Connector_PinHeader_2.54mm:PinHeader_1x04_P2.54mm_Vertical"
 			(at 212.09 90.17 0)
 			(effects

Commit message: Started the floorplan + added the Power LED
Parts:
- U502: footprint Connector_PinHeader_2.54mm:PinHeader_1x04_P2.54mm_Vertical -> ProjectConnectors:SSD1306; Checked E- Da Valutare -> E- Da Valutare-Footprint OK
Changed lines of the file:
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@@
 			)
 		)
-		(property "Footprint" "Connector_PinHeader_2.54mm:PinHeader_1x04_P2.54mm_Vertical"
+		(property "Footprint" "ProjectConnectors:SSD1306"
 			(at 212.09 90.17 0)
 			(effects
@@
 			)
 		)
-		(property "Checked" "E- Da Valutare"
+		(property "Checked" "E- Da Valutare-Footprint OK"
 			(at 227.33 82.55 90)
 			(effects

Commit message: Continued the floor plan
Parts:
- BZ501: footprint ProjectConnectors:Buzzer MLT-7525 -> ProjectConnectors:MLT-8530
Changed lines of the file:
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@@
 			)
 		)
-		(property "Footprint" "ProjectConnectors:Buzzer MLT-7525"
+		(property "Footprint" "ProjectConnectors:MLT-8530"
 			(at 168.275 71.12 90)
 			(effects
