File: POWER_UI.kicad_sch (KiCad schematic)
At the start: 45 parts, among them J601 PWR_IN1, J602 PWR_IN2, J603 PWR_IN3, J604 PWR_IN4, J605 MCP_INT, J606 5V, J607 GND, J608 3V3, J609 EX_PA, J610 EX_PB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

Commit message: routing and silkscreen logo
Other:
- company: Filippo Castellan, Alan Masutti -> Alan Masutti, Filippo Castellan
Changed lines of the file:
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@@
 		(date "2026-03-12")
 		(rev "1.0")
-		(company "Filippo Castellan, Alan Masutti")
+		(company "Alan Masutti, Filippo Castellan")
 	)
 	(rectangle
