File: sensors.kicad_sch (KiCad schematic)
At the start: 44 parts, among them J401 ACC_INT1, J402 BME_SPI, J403 LUX_INT, U202 NUCLEO64-H503RB, U401 LSM6DS3, U402 BME280, U403 OPT4001, U404 INA2180A2, U406 YK16S-L7.2-B10Ka(32-8)-G-A29

Commit message: Continuated routing + fixing SSD1306 footprint
Connections:
- net SHUNT_VDD: no longer JP414.2 (B), JP415.2 (B), U202.78 (VDD), U404.5 (+)
- new net SHUNT_VDD2: JP414.2 (B), JP415.2 (B), U202.78 (VDD), U404.5 (+)
Changed lines of the file:
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@@
 		)
 	)
-	(label "SHUNT_VDD"
+	(label "SHUNT_VDD2"
 		(at 52.07 148.59 0)
 		(effects

Commit message: routing and silkscreen logo
Connections:
- net JOYSTICK_X: now also C410.1, U406.5; no longer C409.1, U406.2
- net JOYSTICK_Y: now also C409.1, U406.2; no longer C410.1, U406.5
Other:
- company: Filippo Castellan, Alan Masutti -> Alan Masutti, Filippo Castellan
Changed lines of the file:
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@@
 		(date "2026-03-12")
 		(rev "1.0")
-		(company "Filippo Castellan, Alan Masutti")
+		(company "Alan Masutti, Filippo Castellan")
 	)
 	(rectangle
@@
 	(hierarchical_label "JOYSTICK_X"
 		(shape output)
-		(at 208.28 124.46 180)
+		(at 245.11 124.46 0)
 		(effects
 			(font
 				(size 1.27 1.27)
 			)
-			(justify right)
+			(justify left)
 		)
 	)
@@
 	(hierarchical_label "JOYSTICK_Y"
 		(shape output)
-		(at 245.11 124.46 0)
+		(at 208.28 124.46 180)
 		(effects
 			(font
 				(size 1.27 1.27)
 			)
-			(justify left)
-		)
-	)
+			(justify right)
+		)
+	)

Commit message: Added pullup to the joystick, Fixes #16
Parts:
- added R408: 5K1, Resistor_SMD:R_0603_1608Metric_Pad0.98x0.95mm_HandSolder, symbol Device:R
- added R409: 10K, Resistor_SMD:R_0603_1608Metric_Pad0.98x0.95mm_HandSolder, symbol Device:R
Connections:
- net +3V3: now also R408.1
- net JOYSTICK_BTN: now also R409.1; no longer C406.1, U406.8
- new net: C406.1, R408.2, R409.2, U406.8
Other:
- moved on the sheet: C406, C409, C410, U406

Commit message: added version marking, generated all the production files, added last connector lcsc number
Parts:
- U202: now not fitted
Changed lines of the file:
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@@
 		(in_bom no)
 		(on_board yes)
-		(dnp no)
+		(dnp yes)
 		(property "Reference" "U202"
 			(at 44.45 107.95 90)
@@
 		(in_bom no)
 		(on_board yes)
-		(dnp no)
+		(dnp yes)
 		(property "Reference" "U202"
 			(at 44.45 148.59 90)
